File: Edurob/Edurob.kicad_sch (KiCad schematic)
At the start: 2 parts

Commit message: Added GPIO Expander, finalized Connector positions
Other:
- added sheet GPIOExpander (gpioExpander.kicad_sch)
Changed lines of the file:
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@@
+    )
+  )
+  (sheet (at 220.98 15.24) (size 26.67 12.7) (fields_autoplaced)
+    (stroke (width 0.1524) (type solid))
+    (fill (color 0 0 0 0.0000))
+    (property "Sheetname" "GPIOExpander" (at 220.98 14.5284 0)
+      (effects (font (size 1.27 1.27)) (justify left bottom))
+    )
+    (property "Sheetfile" "gpioExpander.kicad_sch" (at 220.98 28.5246 0)
+      (effects (font (size 1.27 1.27)) (justify left top))
+    )
+    (instances
+      (project "Edurob"
+        (path "/ea495553-3cd2-4380-af57-b7ab16ec3dc9" (page "9"))
+      )
     )
   )

Commit message: Finished silkscreen + fixed board outline
Parts:
- removed LOGO1: Logo, Footprints:Logo_Cat_15x5, symbol Connector:TestPoint_Small
- removed LOGO2: Logo, Footprints:Logo_Cat_Copper_5x5, symbol Connector:TestPoint_Small
Other:
- added sheet Artwork (artwork.kicad_sch)
Changed lines of the file:
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@@
 (kicad_sch (version 20230121) (generator eeschema)
   (paper "A4")
-  (symbol (lib_id "Connector:TestPoint_Small") (at 15.24 171.45 0) (unit 1)
-    (in_bom yes) (on_board yes) (dnp no)
-    (property "Reference" "LOGO1" (at 17.78 170.18 0)
-      (effects (font (size 1.27 1.27)) (justify left))
-    )
-    (property "Value" "Logo" (at 17.78 172.72 0)
-      (effects (font (size 1.27 1.27)) (justify left))
-    )
-    (property "Footprint" "Footprints:Logo_Cat_15x5" (at 20.32 171.45 0)
-      (effects (font (size 1.27 1.27)) hide)
-    )
-    (property "Datasheet" "~" (at 20.32 171.45 0)
-      (effects (font (size 1.27 1.27)) hide)
-    )
-    (pin "1")
-    (instances
-      (project "DynamixelAdapter"
-        (path "/22517a9a-76da-4fac-8f10-b117f5082986"
-          (reference "LOGO1") (unit 1)
-        )
-      )
-      (project "Edurob"
-        (path "/ea495553-3cd2-4380-af57-b7ab16ec3dc9"
-          (reference "LOGO2") (unit 1)
-        )
-      )
-    )
-  )
-  (symbol (lib_id "Connector:TestPoint_Small") (at 15.24 165.1 0) (unit 1)
-    (in_bom yes) (on_board yes) (dnp no)
-    (property "Reference" "LOGO2" (at 17.78 163.83 0)
-      (effects (font (size 1.27 1.27)) (justify left))
-    )
-    (property "Value" "Logo" (at 17.78 166.37 0)
-      (effects (font (size 1.27 1.27)) (justify left))
-    )
-    (property "Footprint" "Footprints:Logo_Cat_Copper_5x5" (at 20.32 165.1 0)
-      (effects (font (size 1.27 1.27)) hide)
-    )
-    (property "Datasheet" "~" (at 20.32 165.1 0)
-      (effects (font (size 1.27 1.27)) hide)
-    )
-    (pin "1")
-    (instances
-      (project "DynamixelAdapter"
-        (path "/22517a9a-76da-4fac-8f10-b117f5082986"
-          (reference "LOGO2") (unit 1)
-        )
-      )
-      (project "Edurob"
-        (path "/ea495553-3cd2-4380-af57-b7ab16ec3dc9"
-          (reference "LOGO1") (unit 1)
-        )
-      )
-    )
-  )
   (sheet (at 132.08 15.24) (size 30.48 12.7) (fields_autoplaced)
     (stroke (width 0.1524) (type solid))
@@
       )
     )
+  )
+  (sheet (at 248.92 15.24) (size 27.94 12.7) (fields_autoplaced)
+    (stroke (width 0.1524) (type solid))
+    (fill (color 0 0 0 0.0000))
+    (property "Sheetname" "Artwork" (at 248.92 14.5284 0)
+      (effects (font (size 1.27 1.27)) (justify left bottom))
+    )
+    (property "Sheetfile" "artwork.kicad_sch" (at 248.92 28.5246 0)
+      (effects (font (size 1.27 1.27)) (justify left top))
+    )
+    (instances
+      (project "Edurob"
+        (path "/ea495553-3cd2-4380-af57-b7ab16ec3dc9" (page "10"))
+      )
+    )
