File: Edurob/artwork.kicad_sch (KiCad schematic)
At the start: 10 parts

Commit message: Release v1.0.1
Parts:
- LOGO1, LOGO10, LOGO2, LOGO3, LOGO4, LOGO5, LOGO6, LOGO7, LOGO8, LOGO9: Placed (none) -> False
Changed lines of the file:
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@@
+      (effects (font (size 1.27 1.27)) hide)
+    )
+    (property "Placed" "False" (at 74.93 31.75 0)
       (effects (font (size 1.27 1.27)) hide)
     )
@@
       (effects (font (size 1.27 1.27)) hide)
     )
+    (property "Placed" "False" (at 74.93 64.77 0)
+      (effects (font (size 1.27 1.27)) hide)
+    )
     (instances
       (project "Edurob"
@@
       (effects (font (size 1.27 1.27)) hide)
     )
+    (property "Placed" "False" (at 123.19 64.77 0)
+      (effects (font (size 1.27 1.27)) hide)
+    )
     (instances
       (project "Edurob"
@@
   )
   (symbol (lib_id "Graphic:Logo_Open_Hardware_Large") (at 25.4 31.75 0) (unit 1)
-    (in_bom no) (on_board yes) (dnp no) (fields_autoplaced)
+    (in_bom no) (on_board no) (dnp no) (fields_autoplaced)
     (property "Reference" "LOGO5" (at 25.4 19.05 0)
       (effects (font (size 1.27 1.27)) hide)
@@
       (effects (font (size 1.27 1.27)) hide)
     )
+    (property "Placed" "False" (at 25.4 31.75 0)
+      (effects (font (size 1.27 1.27)) hide)
+    )
     (instances
       (project "Edurob"
@@
       (effects (font (size 1.27 1.27)) hide)
     )
+    (property "Placed" "False" (at 123.19 31.75 0)
+      (effects (font (size 1.27 1.27)) hide)
+    )
     (instances
       (project "Edurob"
@@
       (effects (font (size 1.27 1.27)) hide)
     )
+    (property "Placed" "False" (at 50.8 31.75 0)
+      (effects (font (size 1.27 1.27)) hide)
+    )
     (instances
       (project "Edurob"
@@
       (effects (font (size 1.27 1.27)) hide)
     )
+    (property "Placed" "False" (at 99.06 31.75 0)
+      (effects (font (size 1.27 1.27)) hide)
+    )
     (instances
       (project "Edurob"
@@
       (effects (font (size 1.27 1.27)) hide)
     )
+    (property "Placed" "False" (at 99.06 64.77 0)
+      (effects (font (size 1.27 1.27)) hide)
+    )
     (instances
       (project "Edurob"
@@
       (effects (font (size 1.27 1.27)) hide)
     )
+    (property "Placed" "False" (at 50.8 64.77 0)
+      (effects (font (size 1.27 1.27)) hide)
+    )
     (instances
       (project "Edurob"
@@
   )
   (symbol (lib_id "Graphic:Logo_Open_Hardware_Large") (at 25.4 64.77 0) (unit 1)
-    (in_bom no) (on_board yes) (dnp no) (fields_autoplaced)
+    (in_bom no) (on_board no) (dnp no) (fields_autoplaced)
     (property "Reference" "LOGO10" (at 25.4 52.07 0)
       (effects (font (size 1.27 1.27)) hide)
@@
       (effects (font (size 1.27 1.27)) hide)
     )
+    (property "Placed" "False" (at 25.4 64.77 0)
+      (effects (font (size 1.27 1.27)) hide)
+    )
