File: Edurob/controller.kicad_sch (KiCad schematic)
At the start: 9 parts, among them SW1 SW_Push, U4 ESP32-S3-WROOM-1

Commit message: Release v1.0.1
Parts:
- C1: Manufacturer_Name (none) -> TAIYO YUDEN; Manufacturer_Part_Number (none) -> MSASU168SB5105KTNA01; Mouser Part Number (none) -> 963-MSASU168SB5105KT; Mouser Price/Stock (none) -> https://www.mouser.de/ProductDetail/963-MSASU168SB5105KT; Placed (none) -> True
- R2, R36, R37: value 10k -> 10K; Manufacturer_Name (none) -> Vishay / Dale; Manufacturer_Part_Number (none) -> CRCW060310K0FKEA; Mouser Part Number (none) -> 71-CRCW0603-10K-E3; Mouser Price/Stock (none) -> https://www.mouser.de/ProductDetail/71-CRCW0603-10K-E3; Placed (none) -> True
- SW1: Manufacturer_Name (none) -> C&K; Manufacturer_Part_Number (none) -> PTS645VK832LFS; Mouser Part Number (none) -> 611-PTS645VK832; Mouser Price/Stock (none) -> https://www.mouser.de/ProductDetail/611-PTS645VK832; Placed (none) -> False
- U4: Manufacturer_Name (none) -> Espressif Systems; Manufacturer_Part_Number (none) -> ESP32-S3-WROOM-1U-N16R8; Mouser Part Number (none) -> 356-ESP32-S3-WROOM-1U-N16R8; Mouser Price/Stock (none) -> https://www.mouser.de/ProductDetail/356-ESP32S3WM1UN16R8; Placed (none) -> True
Changed lines of the file:
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@@
       (effects (font (size 1.27 1.27)) (justify left))
     )
-    (property "Value" "10k" (at 104.14 176.5299 0)
+    (property "Value" "10K" (at 104.14 176.5299 0)
       (effects (font (size 1.27 1.27)) (justify left))
     )
@@
       (effects (font (size 1.27 1.27)) hide)
     )
+    (property "Manufacturer_Name" "Vishay / Dale" (at 101.6 175.26 0)
+      (effects (font (size 1.27 1.27)) hide)
+    )
+    (property "Manufacturer_Part_Number" "CRCW060310K0FKEA" (at 101.6 175.26 0)
+      (effects (font (size 1.27 1.27)) hide)
+    )
+    (property "Mouser Part Number" "71-CRCW0603-10K-E3" (at 101.6 175.26 0)
+      (effects (font (size 1.27 1.27)) hide)
+    )
+    (property "Mouser Price/Stock" "https://www.mouser.de/ProductDetail/71-CRCW0603-10K-E3" (at 101.6 175.26 0)
+      (effects (font (size 1.27 1.27)) hide)
+    )
+    (property "Placed" "True" (at 101.6 175.26 0)
+      (effects (font (size 1.27 1.27)) hide)
+    )
     (pin "1")
     (pin "2")
@@
     )
     (property "Datasheet" "~" (at 49.53 182.88 0)
+      (effects (font (size 1.27 1.27)) hide)
+    )
+    (property "Manufacturer_Name" "TAIYO YUDEN" (at 49.53 182.88 0)
+      (effects (font (size 1.27 1.27)) hide)
+    )
+    (property "Manufacturer_Part_Number" "MSASU168SB5105KTNA01" (at 49.53 182.88 0)
+      (effects (font (size 1.27 1.27)) hide)
+    )
+    (property "Mouser Part Number" "963-MSASU168SB5105KT" (at 49.53 182.88 0)
+      (effects (font (size 1.27 1.27)) hide)
+    )
+    (property "Mouser Price/Stock" "https://www.mouser.de/ProductDetail/963-MSASU168SB5105KT" (at 49.53 182.88 0)
+      (effects (font (size 1.27 1.27)) hide)
+    )
+    (property "Placed" "True" (at 49.53 182.88 0)
       (effects (font (size 1.27 1.27)) hide)
     )
@@
     )
     (property "Datasheet" "https://www.espressif.com/sites/default/files/documentation/esp32-s3-wroom-1_wroom-1u_datasheet_en.pdf" (at 86.36 135.89 0)
+      (effects (font (size 1.27 1.27)) hide)
+    )
+    (property "Manufacturer_Name" "Espressif Systems" (at 83.82 85.09 0)
+      (effects (font (size 1.27 1.27)) hide)
+    )
+    (property "Manufacturer_Part_Number" "ESP32-S3-WROOM-1U-N16R8" (at 83.82 85.09 0)
+      (effects (font (size 1.27 1.27)) hide)
+    )
+    (property "Mouser Part Number" "356-ESP32-S3-WROOM-1U-N16R8" (at 83.82 85.09 0)
+      (effects (font (size 1.27 1.27)) hide)
+    )
+    (property "Mouser Price/Stock" "https://www.mouser.de/ProductDetail/356-ESP32S3WM1UN16R8" (at 83.82 85.09 0)
+      (effects (font (size 1.27 1.27)) hide)
+    )
+    (property "Placed" "True" (at 83.82 85.09 0)
       (effects (font (size 1.27 1.27)) hide)
     )
@@
       (effects (font (size 1.27 1.27)) (justify left))
     )
-    (property "Value" "10k" (at 52.07 173.9899 0)
+    (property "Value" "10K" (at 52.07 173.9899 0)
       (effects (font (size 1.27 1.27)) (justify left))
     )
@@
     )
     (property "Datasheet" "~" (at 49.53 172.72 0)
+      (effects (font (size 1.27 1.27)) hide)
+    )
+    (property "Manufacturer_Name" "Vishay / Dale" (at 49.53 172.72 0)
+      (effects (font (size 1.27 1.27)) hide)
+    )
+    (property "Manufacturer_Part_Number" "CRCW060310K0FKEA" (at 49.53 172.72 0)
+      (effects (font (size 1.27 1.27)) hide)
+    )
+    (property "Mouser Part Number" "71-CRCW0603-10K-E3" (at 49.53 172.72 0)
+      (effects (font (size 1.27 1.27)) hide)
+    )
+    (property "Mouser Price/Stock" "https://www.mouser.de/ProductDetail/71-CRCW0603-10K-E3" (at 49.53 172.72 0)
+      (effects (font (size 1.27 1.27)) hide)
+    )
+    (property "Placed" "True" (at 49.53 172.72 0)
       (effects (font (size 1.27 1.27)) hide)
     )
@@
       (effects (font (size 1.27 1.27)) hide)
     )
+    (property "Manufacturer_Name" "TAIYO YUDEN" (at 17.78 182.88 0)
+      (effects (font (size 1.27 1.27)) hide)
+    )
+    (property "Manufacturer_Part_Number" "MSASU168SB5105KTNA01" (at 17.78 182.88 0)
+      (effects (font (size 1.27 1.27)) hide)
+    )
+    (property "Mouser Part Number" "963-MSASU168SB5105KT" (at 17.78 182.88 0)
+      (effects (font (size 1.27 1.27)) hide)
+    )
+    (property "Mouser Price/Stock" "https://www.mouser.de/ProductDetail/963-MSASU168SB5105KT" (at 17.78 182.88 0)
+      (effects (font (size 1.27 1.27)) hide)
+    )
+    (property "Placed" "True" (at 17.78 182.88 0)
+      (effects (font (size 1.27 1.27)) hide)
+    )
     (pin "1")
     (pin "2")
@@
       (effects (font (size 1.27 1.27)) (justify left))
     )
-    (property "Value" "10k" (at 20.32 173.9899 0)
+    (property "Value" "10K" (at 20.32 173.9899 0)
       (effects (font (size 1.27 1.27)) (justify left))
     )
@@
     )
     (property "Datasheet" "~" (at 17.78 172.72 0)
+      (effects (font (size 1.27 1.27)) hide)
+    )
+    (property "Manufacturer_Name" "Vishay / Dale" (at 17.78 172.72 0)
+      (effects (font (size 1.27 1.27)) hide)
+    )
+    (property "Manufacturer_Part_Number" "CRCW060310K0FKEA" (at 17.78 172.72 0)
+      (effects (font (size 1.27 1.27)) hide)
+    )
+    (property "Mouser Part Number" "71-CRCW0603-10K-E3" (at 17.78 172.72 0)
+      (effects (font (size 1.27 1.27)) hide)
+    )
+    (property "Mouser Price/Stock" "https://www.mouser.de/ProductDetail/71-CRCW0603-10K-E3" (at 17.78 172.72 0)
+      (effects (font (size 1.27 1.27)) hide)
+    )
+    (property "Placed" "True" (at 17.78 172.72 0)
       (effects (font (size 1.27 1.27)) hide)
     )
@@
       (effects (font (size 1.27 1.27)) (justify left))
     )
-    (property "Value" "10k" (at 113.03 176.5299 0)
+    (property "Value" "10K" (at 113.03 176.5299 0)
       (effects (font (size 1.27 1.27)) (justify left))
     )
@@
     )
     (property "Datasheet" "~" (at 110.49 175.26 0)
+      (effects (font (size 1.27 1.27)) hide)
+    )
+    (property "Manufacturer_Name" "Vishay / Dale" (at 110.49 175.26 0)
+      (effects (font (size 1.27 1.27)) hide)
+    )
+    (property "Manufacturer_Part_Number" "CRCW060310K0FKEA" (at 110.49 175.26 0)
+      (effects (font (size 1.27 1.27)) hide)
+    )
+    (property "Mouser Part Number" "71-CRCW0603-10K-E3" (at 110.49 175.26 0)
+      (effects (font (size 1.27 1.27)) hide)
+    )
+    (property "Mouser Price/Stock" "https://www.mouser.de/ProductDetail/71-CRCW0603-10K-E3" (at 110.49 175.26 0)
+      (effects (font (size 1.27 1.27)) hide)
+    )
+    (property "Placed" "True" (at 110.49 175.26 0)
       (effects (font (size 1.27 1.27)) hide)
     )
@@
     )
     (property "Datasheet" "~" (at 66.04 172.72 0)
+      (effects (font (size 1.27 1.27)) hide)
+    )
+    (property "Manufacturer_Name" "C&K" (at 66.04 177.8 0)
+      (effects (font (size 1.27 1.27)) hide)
+    )
+    (property "Manufacturer_Part_Number" "PTS645VK832LFS" (at 66.04 177.8 0)
+      (effects (font (size 1.27 1.27)) hide)
+    )
+    (property "Mouser Part Number" "611-PTS645VK832" (at 66.04 177.8 0)
+      (effects (font (size 1.27 1.27)) hide)
+    )
+    (property "Mouser Price/Stock" "https://www.mouser.de/ProductDetail/611-PTS645VK832" (at 66.04 177.8 0)
+      (effects (font (size 1.27 1.27)) hide)
+    )
+    (property "Placed" "False" (at 66.04 177.8 0)
       (effects (font (size 1.27 1.27)) hide)
     )
@@
       (effects (font (size 1.27 1.27)) hide)
     )
+    (property "Manufacturer_Name" "C&K" (at 34.29 177.8 0)
+      (effects (font (size 1.27 1.27)) hide)
+    )
+    (property "Manufacturer_Part_Number" "PTS645VK832LFS" (at 34.29 177.8 0)
+      (effects (font (size 1.27 1.27)) hide)
+    )
+    (property "Mouser Part Number" "611-PTS645VK832" (at 34.29 177.8 0)
+      (effects (font (size 1.27 1.27)) hide)
+    )
+    (property "Mouser Price/Stock" "https://www.mouser.de/ProductDetail/611-PTS645VK832" (at 34.29 177.8 0)
+      (effects (font (size 1.27 1.27)) hide)
+    )
+    (property "Placed" "False" (at 34.29 177.8 0)
+      (effects (font (size 1.27 1.27)) hide)
+    )
