File: Edurob/gpioExpander.kicad_sch (KiCad schematic)
At the start: 4 parts, among them IC3 PI4IOE5V6416ZDEX

Commit message: Release v1.0.1
Parts:
- IC3: Height 0.9 -> (none); Mouser Price/Stock https://www.mouser.co.uk/ProductDetail/Diodes-Incorporated/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 -> https://www.mouser.de/ProductDetail/729-PI4IOE5V6416ZDEX; Placed (none) -> True
- JP3: Placed (none) -> False
- R34, R35: value 10k -> 10K; Manufacturer_Name (none) -> Vishay / Dale; Manufacturer_Part_Number (none) -> CRCW060310K0FKEA; Mouser Part Number (none) -> 71-CRCW0603-10K-E3; Mouser Price/Stock (none) -> https://www.mouser.de/ProductDetail/71-CRCW0603-10K-E3; Placed (none) -> True
Changed lines of the file:
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@@
-      (effects (font (size 1.27 1.27)) (justify left top) hide)
-    )
-    (property "Height" "0.9" (at 148.59 464.77 0)
       (effects (font (size 1.27 1.27)) (justify left top) hide)
     )
@@
       (effects (font (size 1.27 1.27)) (justify left top) hide)
     )
-    (property "Mouser Price/Stock" "https://www.mouser.co.uk/ProductDetail/Diodes-Incorporated/PI4IOE5V6416ZDEX?qs=byeeYqUIh0OndNU%2F4OrZvQ%3D%3D" (at 148.59 664.77 0)
+    (property "Mouser Price/Stock" "https://www.mouser.de/ProductDetail/729-PI4IOE5V6416ZDEX" (at 148.59 664.77 0)
       (effects (font (size 1.27 1.27)) (justify left top) hide)
     )
@@
     (property "Manufacturer_Part_Number" "PI4IOE5V6416ZDEX" (at 148.59 864.77 0)
       (effects (font (size 1.27 1.27)) (justify left top) hide)
+    )
+    (property "Placed" "True" (at 121.92 80.01 0)
+      (effects (font (size 1.27 1.27)) hide)
     )
     (pin "3")
@@
       (effects (font (size 1.27 1.27)) hide)
     )
+    (property "Placed" "False" (at 167.64 80.01 0)
+      (effects (font (size 1.27 1.27)) hide)
+    )
     (pin "3")
     (pin "1")
@@
       (effects (font (size 1.27 1.27)) (justify left))
     )
-    (property "Value" "10k" (at 130.81 45.7199 0)
+    (property "Value" "10K" (at 130.81 45.7199 0)
       (effects (font (size 1.27 1.27)) (justify left))
     )
@@
     )
     (property "Datasheet" "~" (at 128.27 44.45 0)
+      (effects (font (size 1.27 1.27)) hide)
+    )
+    (property "Manufacturer_Name" "Vishay / Dale" (at 128.27 44.45 0)
+      (effects (font (size 1.27 1.27)) hide)
+    )
+    (property "Manufacturer_Part_Number" "CRCW060310K0FKEA" (at 128.27 44.45 0)
+      (effects (font (size 1.27 1.27)) hide)
+    )
+    (property "Mouser Part Number" "71-CRCW0603-10K-E3" (at 128.27 44.45 0)
+      (effects (font (size 1.27 1.27)) hide)
+    )
+    (property "Mouser Price/Stock" "https://www.mouser.de/ProductDetail/71-CRCW0603-10K-E3" (at 128.27 44.45 0)
+      (effects (font (size 1.27 1.27)) hide)
+    )
+    (property "Placed" "True" (at 128.27 44.45 0)
       (effects (font (size 1.27 1.27)) hide)
     )
@@
       (effects (font (size 1.27 1.27)) (justify left))
     )
-    (property "Value" "10k" (at 139.7 45.7199 0)
+    (property "Value" "10K" (at 139.7 45.7199 0)
       (effects (font (size 1.27 1.27)) (justify left))
     )
@@
       (effects (font (size 1.27 1.27)) hide)
     )
+    (property "Manufacturer_Name" "Vishay / Dale" (at 137.16 44.45 0)
+      (effects (font (size 1.27 1.27)) hide)
+    )
+    (property "Manufacturer_Part_Number" "CRCW060310K0FKEA" (at 137.16 44.45 0)
+      (effects (font (size 1.27 1.27)) hide)
+    )
+    (property "Mouser Part Number" "71-CRCW0603-10K-E3" (at 137.16 44.45 0)
+      (effects (font (size 1.27 1.27)) hide)
+    )
+    (property "Mouser Price/Stock" "https://www.mouser.de/ProductDetail/71-CRCW0603-10K-E3" (at 137.16 44.45 0)
+      (effects (font (size 1.27 1.27)) hide)
+    )
+    (property "Placed" "True" (at 137.16 44.45 0)
+      (effects (font (size 1.27 1.27)) hide)
+    )
